File: pcb/Y8960_Cartridge/Y8960_Cartridge.kicad_pcb (KiCad board)
At the start: 2 copper layers, 95.2 x 65.4 mm, 61 parts, among them J1 I2S_CONN, J2 SOUNDIN, J3 Conn_02x06_Odd_Even, J4 GND, Q1 NMOS, Q2 NMOS, Q3 NMOS

Commit message: Updated
Parts:
- Q1, Q2, Q3: footprint 0-My_Parts:MOSFET(SMD) -> My Parts:MOSFET(SMD)
- U1: footprint 0-My_Parts:TangPrimer25K(UPPER) -> My Parts:TangPrimer25K(UPPER)
- U3: footprint 0-My_Parts:CLOCK -> My Parts:CLOCK
- U8: footprint 0-My_Parts:QSPI-SRAM 4Mbit (8SOIC) -> My Parts:QSPI-SRAM 4Mbit (8SOIC)
- U9: footprint 0-My_Parts:TangPrimer25K(LOWER) -> My Parts:TangPrimer25K(LOWER)
Connections:
- Q1 pad 2: SLOT_DATA_DIR -> SLOT_BUSDIR
- R20 pad 1: SLOT_DATA_DIR -> SLOT_BUSDIR
Routing:
- net SLOT_BUSDIR: track 26.0 -> 72.3 mm, vias 4 -> 6
- net SLOT_DATA_DIR: track 2.06 -> 0.00 mm
