File: pcb/Y8960_Cartridge/Y8960_Cartridge.kicad_sch (KiCad schematic)
At the start: 59 parts, among them J1 I2S_CONN, J2 SOUNDIN, J3 Conn_02x06_Odd_Even, J4 GND, Q1 NMOS, Q2 NMOS, Q3 NMOS

Commit message: Updated
Connections:
- net SLOT_DATA_DIR is gone; now on net SLOT_BUSDIR: Q1.2 (G), R20.1
Other:
- note added: "/BUSDIR HiZ: Cartridge ← CPU (WRITE) 0: Cartridge → CPU (READ)"
- note added: "SLOT_BUSDIR 0: Cartridge ← CPU (WRITE) 1: Cartridge → CPU (READ)"
- note removed: "/BUSDIR 1: CPU → Cartridge (WRITE) 0: CPU ← Cartridge (READ)"
- note removed: "SLOT_DATA_DIR 0: CPU → Cartridge (WRITE) 1: CPU ← Cartridge (READ)"
Changed lines of the file:
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@@
 		)
 	)
+	(text "SLOT_BUSDIR\n0: Cartridge ← CPU (WRITE)\n1: Cartridge → CPU (READ)"
+		(exclude_from_sim no)
+		(at 250.698 90.424 0)
+		(effects
+			(font
+				(size 1.27 1.27)
+			)
+			(justify left bottom)
+		)
+	)
 	(text "TDI"
 		(exclude_from_sim no)
@@
 		)
 	)
-	(text "SLOT_DATA_DIR\n0: CPU → Cartridge (WRITE)\n1: CPU ← Cartridge (READ)"
+	(text "/BUSDIR\nHiZ: Cartridge ← CPU (WRITE)\n0: Cartridge → CPU (READ)"
 		(exclude_from_sim no)
-		(at 192.278 30.734 0)
+		(at 237.49 23.114 0)
 		(effects
 			(font
@@
 		)
 	)
-	(text "TCK"
+	(text "SLOT_BUSDIR\n0: Cartridge ← CPU (WRITE)\n1: Cartridge → CPU (READ)"
 		(exclude_from_sim no)
-		(at 40.64 245.11 0)
+		(at 192.786 30.988 0)
 		(effects
 			(font
@@
 		)
 	)
-	(text "RX"
+	(text "TCK"
 		(exclude_from_sim no)
-		(at 45.72 247.65 0)
+		(at 40.64 245.11 0)
 		(effects
 			(font
@@
 		)
 	)
-	(text "SLOT_INT : \n1 → /INT=0\n0 or HiZ → /INT=HiZ\n"
+	(text "RX"
 		(exclude_from_sim no)
-		(at 171.958 59.182 0)
+		(at 45.72 247.65 0)
 		(effects
 			(font
@@
 		)
 	)
-	(text "/BUSDIR\n1: CPU → Cartridge (WRITE)\n0: CPU ← Cartridge (READ)"
+	(text "SLOT_INT : \n1 → /INT=0\n0 or HiZ → /INT=HiZ\n"
 		(exclude_from_sim no)
-		(at 233.172 24.13 0)
+		(at 171.958 59.182 0)
 		(effects
 			(font
@@
 		)
 	)
+	(global_label "SLOT_BUSDIR"
+		(shape input)
+		(at 208.28 34.29 180)
+		(fields_autoplaced yes)
+		(effects
+			(font
+				(size 1.27 1.27)
+			)
+			(justify right)
+		)
+		(property "Intersheetrefs" "${INTERSHEET_REFS}"
+			(at 192.8367 34.29 0)
+			(effects
+				(font
+					(size 1.27 1.27)
+				)
+				(justify right)
+				(hide yes)
+			)
+		)
+	)
 	(global_label "SLOT_D4"
 		(shape bidirectional)
@@
 		)
 	)
-	(global_label "SLOT_DATA_DIR"
-		(shape input)
-		(at 208.28 34.29 180)
-		(fields_autoplaced yes)
-		(effects
-			(font
-				(size 1.27 1.27)
-			)
-			(justify right)
-		)
-		(property "Intersheetrefs" "${INTERSHEET_REFS}"
-			(at 191.2643 34.29 0)
-			(effects
-				(font
-					(size 1.27 1.27)
-				)
-				(justify right)
-				(hide yes)
-			)
-		)
-	)
 	(global_label "A15"
 		(shape output)
@@
 		)
 		(instances
-			(project ""
+			(project "Y8960_Cartridge"
 				(path "/0daedcdd-be04-453f-bcf7-9a74be29633a"
 					(reference "D1")
@@
 		)
 		(instances
-			(project ""
+			(project "Y8960_Cartridge"
 				(path "/0daedcdd-be04-453f-bcf7-9a74be29633a"
 					(reference "U3")
@@
 		)
 		(instances
-			(project ""
+			(project "Y8960_Cartridge"
 				(path "/0daedcdd-be04-453f-bcf7-9a74be29633a"
 					(reference "U9")
@@
 		)
 		(instances
-			(project ""
+			(project "Y8960_Cartridge"
 				(path "/0daedcdd-be04-453f-bcf7-9a74be29633a"
 					(reference "R1")
@@
 		)
 		(instances
-			(project ""
+			(project "Y8960_Cartridge"
 				(path "/0daedcdd-be04-453f-bcf7-9a74be29633a"
 					(reference "#PWR01")
@@
 		)
 		(instances
-			(project ""
+			(project "Y8960_Cartridge"
 				(path "/0daedcdd-be04-453f-bcf7-9a74be29633a"
 					(reference "#PWR05")
@@
 		)
 		(instances
-			(project ""
+			(project "Y8960_Cartridge"
 				(path "/0daedcdd-be04-453f-bcf7-9a74be29633a"
 					(reference "C1")
@@
 		)
 		(instances
-			(project ""
+			(project "Y8960_Cartridge"
 				(path "/0daedcdd-be04-453f-bcf7-9a74be29633a"
 					(reference "#FLG02")
@@
 		)
 		(instances
-			(project ""
+			(project "Y8960_Cartridge"
 				(path "/0daedcdd-be04-453f-bcf7-9a74be29633a"
 					(reference "#FLG01")
@@
 		)
 		(instances
-			(project ""
+			(project "Y8960_Cartridge"
 				(path "/0daedcdd-be04-453f-bcf7-9a74be29633a"
 					(reference "U2")
@@
 		)
 		(instances
-			(project ""
+			(project "Y8960_Cartridge"
 				(path "/0daedcdd-be04-453f-bcf7-9a74be29633a"
 					(reference "U1")
@@
 		)
 		(instances
-			(project ""
+			(project "Y8960_Cartridge"
 				(path "/0daedcdd-be04-453f-bcf7-9a74be29633a"
 					(reference "J2")
@@
 		)
 		(instances
-			(project ""
+			(project "Y8960_Cartridge"
 				(path "/0daedcdd-be04-453f-bcf7-9a74be29633a"
 					(reference "J1")
@@
 		)
 		(instances
-			(project ""
+			(project "Y8960_Cartridge"
 				(path "/0daedcdd-be04-453f-bcf7-9a74be29633a"
 					(reference "U4")
@@
 		)
 		(instances
-			(project ""
+			(project "Y8960_Cartridge"
 				(path "/0daedcdd-be04-453f-bcf7-9a74be29633a"
 					(reference "U8")
@@
 		)
 		(instances
-			(project ""
+			(project "Y8960_Cartridge"
 				(path "/0daedcdd-be04-453f-bcf7-9a74be29633a"
 					(reference "#PWR02")
